File: brew_HW_stm8s207.kicad_pcb (KiCad board)
At the start: 2 copper layers, 199.4 x 97.8 mm, 175 parts, among them CON1 24V DC IN, CON10 THLT, CON11 TMLT, CON12 OW1-4X, CON13 OW2-4X, CON14 L3-DET, CON15 FLOWS, CON16 FLOW_C, CON17 FLOW_D, CON18 FREE_IO, CON19 UART, CON2 Serial Bus, CON20 DBG, CON21 FLOWS, CON22 V1, CON23 V2, CON24 V3, CON25 V4, CON26 V5, CON27 V6, CON28 V7, CON29 V8, CON3 Wiz550io, CON4 L2-DET, CON5 FP_LEDS, CON6 PWM24V, CON7 LM35, CON8 230V_OUT, CON9 SSR_ELE_HTR, K1 G5V1-24, K2 G5V1-24, K3 G5V1-24, K4 G5V1-24, K5 G5V1-24, K6 G5V1-24, K7 G5V1-24, K8 G5V1-24, Q1 BSS138, Q2 BC847, Q3 BCP53, Q4 BCP53, SW1 Reset Switch, U1 LM7805, U10 LM393, U2 LD1117V33, U3 LM7805, U4 STM8S207R8, U5 DS2482, U6 DS2482, U7 DS2482, U8 DS2482, U9 TD62783A, Y1 24 MHz

Commit message: Brew HW R4.30 kicad files
Parts:
- removed CON14: L3-DET, Library_Emile:AK500_2
- removed CON15: FLOWS, Connector_PinSocket_2.54mm:PinSocket_1x05_P2.54mm_Vertical
- removed CON19: UART, Connector_PinSocket_2.54mm:PinSocket_2x03_P2.54mm_Vertical
- removed CON4: L2-DET, Library_Emile:AK500_2
- added C37: 100n, Capacitor_SMD:C_1206_3216Metric, B.Cu at (213.6, 73.7)
- added C39: 10u, Capacitor_THT:CP_Radial_D5.0mm_P2.00mm, F.Cu at (213.9, 70.9)
- added C7: 100n, Capacitor_SMD:C_1206_3216Metric, B.Cu at (200.2, 145.9)
- added J14: PHASE DETECT, Connector_PinSocket_2.54mm:PinSocket_1x04_P2.54mm_Vertical, F.Cu at (195.1, 149.6)
- added J15: FLOW, Library_Emile:PS2-MINI-DIN6, F.Cu at (196.1, 54.8)
- added J19: UART, Connector_PinSocket_2.54mm:PinSocket_1x03_P2.54mm_Vertical, F.Cu at (146.5, 118.0)
- added J30: WATER LEVEL, Connector_PinSocket_2.54mm:PinSocket_1x04_P2.54mm_Vertical, F.Cu at (207.8, 149.6)
- added J4: W5500_Lite, Library_Emile:W55000_Lite, F.Cu at (171.1, 67.5)
- added R51: 10R, Resistor_SMD:R_1206_3216Metric, B.Cu at (209.4, 72.2)
- added TP10: scl2, TestPoint:TestPoint_Pad_D1.0mm, F.Cu at (150.7, 68.0)
- added TP11: sda1, TestPoint:TestPoint_Pad_D1.0mm, F.Cu at (141.6, 67.8)
- added TP12: scl1, TestPoint:TestPoint_Pad_D1.0mm, F.Cu at (144.6, 67.9)
- added TP13: bz, TestPoint:TestPoint_Pad_D1.0mm, F.Cu at (179.6, 133.0)
- added TP14: osci, TestPoint:TestPoint_Pad_D1.0mm, F.Cu at (144.5, 106.6)
- added TP15: 1V07, TestPoint:TestPoint_Pad_D1.0mm, F.Cu at (111.9, 121.1)
- added TP8: Vcap, TestPoint:TestPoint_Pad_D1.0mm, F.Cu at (152.5, 105.0)
- added TP9: sda2, TestPoint:TestPoint_Pad_D1.0mm, F.Cu at (147.8, 68.0)
- C1, C12, C15, C2, C28, C4: footprint Capacitor_THT:CP_Radial_D14.0mm_P7.50mm -> Capacitor_THT:CP_Radial_D12.5mm_P5.00mm
- J12: renamed from CON12; value OW1-4X -> OW4X
- J13: renamed from CON13; value OW2-4X -> OW4X
- J16: renamed from CON16; value FLOW_C -> FLOW
- J17: renamed from CON17; value FLOW_D -> FLOW
- Q3, Q4: footprint Package_TO_SOT_SMD:SOT-223-3_TabPin2 -> Package_TO_SOT_SMD:SOT-223
- R38: value 60R -> 47R
- R39: moved to F.Cu
- SW1: value Reset Switch -> RESET
- TH1, TH2, TH3, TH4, TH5, TH6, TH7, TH8: footprint Resistor_THT:R_Radial_Power_L11.0mm_W7.0mm_P5.00mm -> Resistor_THT:R_Box_L8.4mm_W2.5mm_P5.08mm
- TP7: value GND -> Vref; footprint Library_Emile:TestPoint_Loop_D2.54mm_Drill1.5mm_Beaded -> TestPoint:TestPoint_Pad_D1.0mm
- moved TP7 17.5 mm to (152.4, 108.7)
- moved R50 15.1 mm to (206.3, 72.2)
- moved R49 14.7 mm to (202.9, 72.2)
- moved J3 14.5 mm to (169.5, 84.2), turned to -90 degrees
- moved R48 14.3 mm to (199.5, 72.1)
- moved R47 13.9 mm to (196.1, 72.2)
- moved C17 8.10 mm to (109.0, 125.9), turned to -90 degrees
- moved C11 5.62 mm to (112.0, 103.3), turned to -90 degrees
- moved C27 5.46 mm to (105.8, 93.8), turned to -90 degrees
- moved C33 5.33 mm to (220.2, 73.7)
- moved R39 5.09 mm to (141.0, 82.1), turned to -90 degrees
- moved BZ1 4.67 mm to (204.8, 118.2)
- moved C35 4.50 mm to (220.5, 70.8)
- moved C29 3.96 mm to (95.9, 108.5)
- moved C12 1.77 mm to (204.2, 127.8)
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- renumbered CON1 to J1, CON10 to J10, CON11 to J11, CON18 to J18, CON2 to J2, CON20 to J20, CON21 to J21, CON22 to J22, CON23 to J23, CON24 to J24, CON25 to J25, CON26 to J26, CON27 to J27, CON28 to J28, CON29 to J29, CON3 to J3, CON5 to J5, CON6 to J6, CON7 to J7, CON8 to J8, CON9 to J9
Connections:
- D8 pad 1: Net-(CON6-Pin_2) -> Net-(D8-K)
- D9 pad 1: Net-(CON6-Pin_4) -> Net-(D9-K)
- J6 pad 2: Net-(CON6-Pin_2) -> Net-(D8-K)
- J6 pad 4: Net-(CON6-Pin_4) -> Net-(D9-K)
- Q3 pad 2: Net-(CON6-Pin_4) -> Net-(D9-K)
- Q4 pad 2: Net-(CON6-Pin_2) -> Net-(D8-K)
- R28 pad 2: Net-(CON6-Pin_4) -> Net-(D9-K)
- R33 pad 2: Net-(CON6-Pin_2) -> Net-(D8-K)
Routing:
- net /STM8S207 Microcontroller/RX3: track 22.1 -> 118.9 mm, vias 0 -> 2
- net /STM8S207 Microcontroller/TX3: track 26.1 -> 117.6 mm, vias 0 -> 2
- net Net-(D8-K): track 0.00 -> 48.0 mm, vias 0 -> 2
- net Net-(CON6-Pin_2): track 48.0 -> 0.00 mm, vias 2 -> 0
- net /Power Supply +24V, +7 Vdc, +5Vdc, +3V3/+3V3: track 226.8 -> 260.7 mm, vias 10 -> 12
- net Net-(J15-Pin_6): track 0.00 -> 31.3 mm, vias 0 -> 1
- net /STM8S207 Microcontroller/L2DET: track 152.6 -> 122.0 mm
- net Net-(D9-K): track 0.00 -> 30.4 mm, vias 0 -> 1
- net Net-(CON6-Pin_4): track 30.4 -> 0.00 mm, vias 1 -> 0
- net /STM8S207 Microcontroller/~{SPI_RST}: track 72.7 -> 102.6 mm, vias 2 -> 3
- net /STM8S207 Microcontroller/MISO_3V3: track 13.4 -> 43.0 mm, vias 2 -> 3
- net /STM8S207 Microcontroller/SPI_MOSI: track 155.4 -> 178.9 mm, vias 2 -> 4
- net VCC: track 572.4 -> 591.9 mm
- net /STM8S207 Microcontroller/SPI_CLK: track 159.5 -> 173.5 mm
- net /Digital IO and Connectors/SCL2: track 92.3 -> 104.8 mm, vias 2 -> 4
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Other:
- board text added: "+3V3"
- board text added: "+5VE"
- board text added: "0 0"
- board text added: "0 1"
- board text added: "1 0"
- board text added: "1 1"
- board text added: "BK_PWM"
- board text added: "BREW HW v4.30 Emile 09-'26"
- board text added: "HLT_PWM"
- board text added: "L2"
- board text added: "L3"
- board text added: "PHASE- DETECT"
- board text added: "RX3"
- board text added: "TX3"
- board text removed: "BREW HW v4.21 Emile 08-'26"
- board text removed: "GND L2"
- board text removed: "GND L3"
- board text removed: "RX3 TX3 GND"
