File: brew_HW_stm8s207_1.kicad_sch (KiCad schematic)
At the start: 47 parts, among them CON14 L3-DET, CON18 FREE_IO, CON19 UART, CON2 Serial Bus, CON20 DBG, CON3 Wiz550io, CON4 L2-DET, CON5 FP_LEDS, CON7 LM35, CON8 230V_OUT, CON9 SSR_ELE_HTR, Q1 BSS138, Q2 BC847, SW1 Reset Switch, U4 STM8S207R8, Y1 24 MHz

Commit message: Brew HW R4.30 kicad files
Parts:
- removed CON14: L3-DET, Library_Emile:AK500_2, symbol Connector:Conn_01x02_Socket
- removed CON19: UART, Connector_PinSocket_2.54mm:PinSocket_2x03_P2.54mm_Vertical, symbol Connector_Generic:Conn_02x03_Odd_Even
- removed CON4: L2-DET, Library_Emile:AK500_2, symbol Connector:Conn_01x02_Socket
- added C7: 100n, Capacitor_SMD:C_1206_3216Metric, symbol Device:C
- added J14: PHASE DETECT, Connector_PinSocket_2.54mm:PinSocket_1x04_P2.54mm_Vertical, symbol Connector_Generic:Conn_01x04
- added J19: UART, Connector_PinSocket_2.54mm:PinSocket_1x03_P2.54mm_Vertical, symbol Connector_Generic:Conn_01x03
- added J30: WATER LEVEL, Connector_PinSocket_2.54mm:PinSocket_1x04_P2.54mm_Vertical, symbol Connector_Generic:Conn_01x04
- added J4: W5500_Lite, Library_Emile:W55000_Lite, symbol Emile_Custom:W5500_Lite
- added TP10: scl2, TestPoint:TestPoint_Pad_D1.0mm, symbol Connector:TestPoint
- added TP11: sda1, TestPoint:TestPoint_Pad_D1.0mm, symbol Connector:TestPoint
- added TP12: scl1, TestPoint:TestPoint_Pad_D1.0mm, symbol Connector:TestPoint
- added TP13: bz, TestPoint:TestPoint_Pad_D1.0mm, symbol Connector:TestPoint
- added TP14: osci, TestPoint:TestPoint_Pad_D1.0mm, symbol Connector:TestPoint
- added TP8: Vcap, TestPoint:TestPoint_Pad_D1.0mm, symbol Connector:TestPoint
- added TP9: sda2, TestPoint:TestPoint_Pad_D1.0mm, symbol Connector:TestPoint
- R38: value 60R -> 47R
- SW1: value Reset Switch -> RESET
- TP7: value GND -> Vref; footprint Library_Emile:TestPoint_Loop_D2.54mm_Drill1.5mm_Beaded -> TestPoint:TestPoint_Pad_D1.0mm
- renumbered CON18 to J18, CON2 to J2, CON20 to J20, CON3 to J3, CON5 to J5, CON7 to J7, CON8 to J8, CON9 to J9
Connections:
- net +3V3: now also J4.6 (3V3D)
- net BUZZER: now also TP13.1
- net GND: now also C7.2, J14.1 (Pin_1), J14.3 (Pin_3), J19.3 (Pin_3), J30.3 (Pin_3), J4.1 (GND)
- net L2DET: now also J14.4 (Pin_4)
- net L3DET: now also J14.2 (Pin_2)
- net MISO_3V3: now also J4.3 (MISO)
- net OSCI: now also TP14.1
- net RX1: now also J19.1 (Pin_1)
- net RX3: now also J30.1 (Pin_1)
- net SCL1: now also TP12.1
- net SCL2: now also TP10.1
- net SDA1: now also TP11.1
- net SDA2: now also TP9.1
- net SPI_CLK: now also J4.4 (SCLK)
- net SPI_MOSI: now also J4.2 (MOSI)
- net TX1: now also J19.2 (Pin_2)
- net TX3: now also J30.2 (Pin_2)
- net VCC: now also C7.1, J30.4 (Pin_4)
- net ~{SPI_RST}: now also J4.9 (~{RST})
- net ~{SPI_SS}: now also J4.5 (~{SCS})
- net at C50.1, U4.6 (VCAP): now also TP8.1
- no-connect marks 3 -> 5
Other:
- note added: "A02YYUW Ultrasonic Sensor with UART output. Note: RX - TX3 and TX - RX3."
- note added: "Detection of 2nd and 3rd power phases, phase 1 powers PCB."
- note added: "Ethernet Connector W5500-Lite PCB"
- note added: "Ethernet Connector WIZ550io PCB"
- note added: "FLOW1: HLT->MLT Flowsensor FLOW2: MLT->Boil Flowsensor FLOW3: CFC out Flowsensor FLOW4: Flowsensor optional ADC6 : LM35 Temperature Sensor"
- note added: "Free IO pins"
- note added: "Frontpanel LEDs MAX7219"
- note added: "LM35 Temp. sensor"
- note added: "SWIM connector"
- note added: "UART Debugging Output"
- note removed: "FLOW1: HLT->MLT Flowsensor FLOW2: MLT->Boil Flowsensor FLOW3: CFC out Flowsensor FLOW4: Flowsensor optional ADC6: LM35 Temperature Sensor"
- title: (none) -> Brew Hardware STM8S207R8
- moved on the sheet: C6, J7, R21
