File: brew_HW_stm8s207_2.kicad_sch (KiCad schematic)
At the start: 36 parts, among them U1 LM7805, U10 LM393, U2 LD1117V33, U3 LM7805

Commit message: Brew HW R4.30 kicad files
Parts:
- C1, C12, C15, C2, C28, C4: footprint Capacitor_THT:CP_Radial_D14.0mm_P7.50mm -> Capacitor_THT:CP_Radial_D12.5mm_P5.00mm
Other:
- title: (none) -> Brew Hardware STM8S207R8
Changed lines of the file:
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@@
 	(generator_version "10.0")
 	(paper "A4")
+	(title_block
+		(title "Brew Hardware STM8S207R8")
+		(date "2026-09-27")
+		(rev "R4.30")
+	)
 	(text "This +5V power-supply is needed\nfor external devices (e.g. temp. sensors)."
 		(exclude_from_sim no)
@@
 			)
 		)
-		(property "Footprint" "Capacitor_THT:CP_Radial_D14.0mm_P7.50mm"
+		(property "Footprint" "Capacitor_THT:CP_Radial_D12.5mm_P5.00mm"
 			(at 63.1952 53.34 0)
 			(hide yes)
@@
 			)
 		)
-		(property "Footprint" "Capacitor_THT:CP_Radial_D14.0mm_P7.50mm"
+		(property "Footprint" "Capacitor_THT:CP_Radial_D12.5mm_P5.00mm"
 			(at 93.6752 53.34 0)
 			(hide yes)
@@
 		)
 		(property "Value" "1000u"
-			(at 35.56 49.53 0)
+			(at 40.64 49.53 0)
 			(show_name no)
 			(do_not_autoplace no)
@@
 			)
 		)
-		(property "Footprint" "Capacitor_THT:CP_Radial_D14.0mm_P7.50mm"
+		(property "Footprint" "Capacitor_THT:CP_Radial_D12.5mm_P5.00mm"
 			(at 50.4952 53.34 0)
 			(hide yes)
@@
 			)
 		)
-		(property "Footprint" "Capacitor_THT:CP_Radial_D14.0mm_P7.50mm"
+		(property "Footprint" "Capacitor_THT:CP_Radial_D12.5mm_P5.00mm"
 			(at 167.3352 46.99 0)
 			(hide yes)
@@
 			)
 		)
-		(property "Footprint" "Capacitor_THT:CP_Radial_D14.0mm_P7.50mm"
+		(property "Footprint" "Capacitor_THT:CP_Radial_D12.5mm_P5.00mm"
 			(at 167.3352 77.47 0)
 			(hide yes)
@@
 			)
 		)
-		(property "Footprint" "Capacitor_THT:CP_Radial_D14.0mm_P7.50mm"
+		(property "Footprint" "Capacitor_THT:CP_Radial_D12.5mm_P5.00mm"
 			(at 167.3352 110.49 0)
 			(hide yes)
