File: brew_HW_stm8s207_3.kicad_sch (KiCad schematic)
At the start: 88 parts, among them CON10 THLT, CON11 TMLT, CON12 OW1-4X, CON13 OW2-4X, CON15 FLOWS, CON16 FLOW_C, CON17 FLOW_D, CON21 FLOWS, CON22 V1, CON23 V2, CON24 V3, CON25 V4, CON26 V5, CON27 V6, CON28 V7, CON29 V8, CON6 PWM24V, K1 G5V1-24, K2 G5V1-24, K3 G5V1-24, K4 G5V1-24, K5 G5V1-24, K6 G5V1-24, K7 G5V1-24, K8 G5V1-24, Q3 BCP53, Q4 BCP53, U10 LM393, U5 DS2482, U6 DS2482, U7 DS2482, U8 DS2482, U9 TD62783A

Commit message: Brew HW R4.30 kicad files
Parts:
- removed CON15: FLOWS, Connector_PinSocket_2.54mm:PinSocket_1x05_P2.54mm_Vertical, symbol Connector_Generic:Conn_01x05
- added C37: 100n, Capacitor_SMD:C_1206_3216Metric, symbol Device:C
- added C39: 10u, Capacitor_THT:CP_Radial_D5.0mm_P2.00mm, symbol Device:C_Polarized
- added J15: FLOW, Library_Emile:PS2-MINI-DIN6, symbol Connector_Generic:Conn_01x06
- added R51: 10R, Resistor_SMD:R_1206_3216Metric, symbol Device:R
- added TP15: 1V07, TestPoint:TestPoint_Pad_D1.0mm, symbol Connector:TestPoint
- J12: renamed from CON12; value OW1-4X -> OW4X
- J13: renamed from CON13; value OW2-4X -> OW4X
- J16: renamed from CON16; value FLOW_C -> FLOW
- J17: renamed from CON17; value FLOW_D -> FLOW
- Q3, Q4: footprint Package_TO_SOT_SMD:SOT-223-3_TabPin2 -> Package_TO_SOT_SMD:SOT-223
- TH1, TH2, TH3, TH4, TH5, TH6, TH7, TH8: footprint Resistor_THT:R_Radial_Power_L11.0mm_W7.0mm_P5.00mm -> Resistor_THT:R_Box_L8.4mm_W2.5mm_P5.08mm
- renumbered CON10 to J10, CON11 to J11, CON21 to J21, CON22 to J22, CON23 to J23, CON24 to J24, CON25 to J25, CON26 to J26, CON27 to J27, CON28 to J28, CON29 to J29, CON6 to J6
Connections:
- net +5V_EXT: now also R51.1
- net 1.07V: now also TP15.1
- net FLOW1: now also J15.2 (Pin_2)
- net FLOW2: now also J15.3 (Pin_3)
- net FLOW3: now also J15.4 (Pin_4)
- net FLOW4: now also J15.5 (Pin_5)
- net GND: now also C37.2, C39.2, J15.1 (Pin_1)
- new net: C37.1, C39.1, J15.6 (Pin_6), R51.2
Other:
- note added: "J10 and J11 Temperature Sensors I2C (LM92) or One-Wire (DS18B20)"
- note added: "J12 and J13 Temperature Sensors 4 x One-Wire"
- note removed: "CON10 and CON11 Temperature Sensors I2C (LM92) or One-Wire (DS18B20)"
- note removed: "CON12 and CON13 Temperature Sensors 4 x One-Wire"
- title: (none) -> Brew Hardware STM8S207R8
- moved on the sheet: J21, R47, R48, R49, R50
